File: OperationBaldr.kicad_pcb (KiCad board)
At the start: 2 copper layers, 80 x 100 mm, 20 parts, among them J1 Conn_01x10_Pin, J2 Conn_01x04_Pin, U4 ULN2003A, U5 ULN2003A, U6 74HC595, U7 74HC595, U8 74HC595, U9 ULN2003A

Commit message: Added cad directory
Added cad directory with casing step file. Also made a minor
schematic revision (adding values to the resistor networks).
Parts:
- RN1, RN2, RN3: value R_Network08 -> 10k
Changed lines of the file:
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@@
 			)
 		)
-		(property "Value" "R_Network08"
+		(property "Value" "10k"
 			(at 11.43 2.4 0)
 			(layer "F.Fab")
@@
 			)
 		)
-		(property "Value" "R_Network08"
+		(property "Value" "10k"
 			(at 11.43 2.4 0)
 			(layer "F.Fab")
@@
 			)
 		)
-		(property "Value" "R_Network08"
+		(property "Value" "10k"
 			(at 11.43 2.4 0)
 			(layer "F.Fab")
