File: cad/pcb/OperationBaldr.kicad_pcb (KiCad board)
At the start: 2 copper layers, 80 x 100 mm, 20 parts, among them J1 Conn_01x10_Pin, J2 Conn_01x04_Pin, U4 ULN2003A, U5 ULN2003A, U6 74HC595, U7 74HC595, U8 74HC595, U9 ULN2003A

Commit message: Added embedded rust code
Added an embedded rust program to control the device.
Also restructered file hierarchy, and made revisions to schematic/pcb.
Connections:
- U4 pad 9: GND -> unconnected-(U4-COM-Pad9)
- U5 pad 9: GND -> unconnected-(U5-COM-Pad9)
- U9 pad 9: GND -> unconnected-(U9-COM-Pad9)
Changed lines of the file:
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@@
 	(title_block
 		(title "Baldr PCB")
-		(date "2024-06-18")
-		(rev "0.1.0")
+		(date "2024-08-28")
+		(rev "0.1.1")
 	)
 	(layers
@@
 	(net 97 "/SW_GND")
 	(net 98 "/SW_3V3")
+	(net 99 "unconnected-(U4-COM-Pad9)")
+	(net 100 "unconnected-(U5-COM-Pad9)")
+	(net 101 "unconnected-(U9-COM-Pad9)")
 	(footprint "Custom:STM32_blackpill"
 		(layer "F.Cu")
@@
 			(layers "*.Cu" "*.Mask")
 			(remove_unused_layers no)
-			(net 1 "GND")
+			(net 99 "unconnected-(U4-COM-Pad9)")
 			(pinfunction "COM")
-			(pintype "passive")
+			(pintype "passive+no_connect")
 		)
 		(pad "10" thru_hole oval
@@
 			(layers "*.Cu" "*.Mask")
 			(remove_unused_layers no)
-			(net 1 "GND")
+			(net 100 "unconnected-(U5-COM-Pad9)")
 			(pinfunction "COM")
-			(pintype "passive")
+			(pintype "passive+no_connect")
 		)
 		(pad "10" thru_hole oval
@@
 			(layers "*.Cu" "*.Mask")
 			(remove_unused_layers no)
-			(net 1 "GND")
+			(net 101 "unconnected-(U9-COM-Pad9)")
 			(pinfunction "COM")
-			(pintype "passive")
+			(pintype "passive+no_connect")
 		)
 		(pad "10" thru_hole oval
